Commit message: Update robot xacro files

File: parc_robot_description/urdf/d435.xacro (robot description, xacro)
@@ -6,12 +6,5 @@
   <xacro:property name="d435_cam_depth_to_infra2_offset" value="-0.050"/>
   <xacro:property name="d435_cam_depth_to_color_offset" value="0.015"/>
-  <!-- Sensor image dimensions -->
-  <xacro:property name="color_width" value="1280"/>
-  <xacro:property name="color_height" value="720"/>
-  <xacro:property name="infra_width" value="640"/>
-  <xacro:property name="infra_height" value="480"/>
-  <xacro:property name="depth_width" value="1280"/>
-  <xacro:property name="depth_height" value="720"/>
-    <!-- D435 camera link -->
+  <!-- D435 camera link -->
     <link name="${name}_link">
       <visual>
@@ -33,11 +26,18 @@
       </xacro:unless>
     </joint>
-    <!-- D435 optical link -->
+    <!-- D435 camera depth link and joint -->
+    <link name="${name}_depth"></link>
+    <joint name="${name}_depth_joint" type="fixed">
+      <origin xyz="0 0 0" rpy="0 0 0" />
+      <parent link="${name}_link"/>
+      <child link="${name}_depth"/>
+    </joint>
+    <!-- D435 depth optical link and joint -->
     <link name="${name}_depth_optical_frame"></link>
     <!-- D435 camera optical joint -->
-    <joint name="${name}_depth_joint" type="fixed">
-      <parent link="${name}_link"/>
+    <joint name="${name}_depth_optical_joint" type="fixed">
+      <origin xyz="0.0 0.0 0.0" rpy="-${pi/2} 0 -${pi/2}"/>
+      <parent link="${name}_depth"/>
       <child link="${name}_depth_optical_frame"/>
-      <origin rpy="-${pi/2} 0 -${pi/2}" xyz="0.0 0.0 0.0"/>
     </joint>
     <!-- Camera left IR joints and links -->
@@ -50,5 +50,5 @@
     <link name="${name}_infra1_optical_frame"/>
     <joint name="${name}_infra1_optical_joint" type="fixed">
-      <origin xyz="0 0 0" rpy="-${pi/2} 0 -${pi/2}"/>
+      <origin xyz="0.0 0.0 0.0" rpy="-${pi/2} 0 -${pi/2}"/>
       <parent link="${name}_infra1_frame"/>
       <child link="${name}_infra1_optical_frame"/>
@@ -63,9 +63,9 @@
     <link name="${name}_infra2_optical_frame"/>
     <joint name="${name}_infra2_optical_joint" type="fixed">
-      <origin xyz="0 0 0" rpy="-${pi/2} 0 -${pi/2}"/>
+      <origin xyz="0.0 0.0 0.0" rpy="-${pi/2} 0 -${pi/2}"/>
       <parent link="${name}_infra2_frame"/>
       <child link="${name}_infra2_optical_frame"/>
     </joint>
-    <!-- Camera color joints and links -->
+    <!-- Camera color joint and link -->
     <link name="${name}_color_frame"/>
     <joint name="${name}_color_joint" type="fixed">
@@ -80,13 +80,19 @@
       <child link="${name}_color_optical_frame"/>
     </joint>
-    <gazebo reference="${name}">
-      <sensor name="${name}_color" type="camera">
-        <camera name="${name}">
+    <!-- Gazebo color frame link reference -->
+    <gazebo reference="${name}_color_frame">
+      <sensor type="camera" name="${name}_color">
+        <always_on>true</always_on>
+        <visualize>false</visualize>
+        <update_rate>30.0</update_rate>
+        <topic>${name}_color/image_raw</topic>
+        <gz_frame_id>${name}_color_optical_frame</gz_frame_id>
+        <camera name="${name}_color">
           <camera_info_topic>${name}_color/camera_info</camera_info_topic>
           <horizontal_fov>1.57</horizontal_fov>
           <image>
-            <width>${color_width}</width>
-            <height>${color_height}</height>
-            <format>RGB_INT8</format>
+            <width>640</width>
+            <height>480</height>
+            <format>R8G8B8</format>
           </image>
           <clip>
@@ -100,68 +106,21 @@
           </noise>
         </camera>
+      </sensor>
+    </gazebo>
+    <!-- Gazebo depth camera link reference -->
+    <gazebo reference="${name}_depth">
+      <sensor type="rgbd_camera" name="${name}_depth">
         <always_on>true</always_on>
-        <visualize>true</visualize>
-        <update_rate>30</update_rate>
-        <topic>${name}_color/image_raw</topic>
-        <gz_frame_id>${name}_color_optical_frame</gz_frame_id>
-      </sensor>
-      <sensor name="${name}_infra1" type="camera">
-        <camera name="${name}">
-          <camera_info_topic>${name}_infra1/camera_info</camera_info_topic>
-          <horizontal_fov>1.57</horizontal_fov>
-          <image>
-            <width>${infra_width}</width>
-            <height>${infra_height}</height>
-            <format>L_INT8</format>
-          </image>
-          <clip>
-            <near>0.1</near>
-            <far>100</far>
-          </clip>
-          <noise>
-            <type>gaussian</type>
-            <mean>0.0</mean>
-            <stddev>0.05</stddev>
-          </noise>
-        </camera>
-        <always_on>false</always_on>
         <visualize>false</visualize>
-        <update_rate>30</update_rate>
-        <topic>${name}_infra1/image_raw</topic>
-        <gz_frame_id>${name}_infra1_optical_frame</gz_frame_id>
-      </sensor>
-      <sensor name="${name}_infra2" type="camera">
-        <camera name="${name}">
-          <camera_info_topic>${name}_infra2/camera_info</camera_info_topic>
-          <horizontal_fov>1.57</horizontal_fov>
-          <image>
-            <width>${infra_width}</width>
-            <height>${infra_height}</height>
-            <format>L_INT8</format>
-          </image>
-          <clip>
-            <near>0.1</near>
-            <far>100</far>
-          </clip>
-          <noise>
-            <type>gaussian</type>
-            <mean>0.0</mean>
-            <stddev>0.05</stddev>
-          </noise>
-        </camera>
-        <always_on>false</always_on>
-        <visualize>false</visualize>
-        <update_rate>30</update_rate>
-        <topic>${name}_infra1/image_raw</topic>
-        <gz_frame_id>${name}_infra2_optical_frame</gz_frame_id>
-      </sensor>
-      <!-- <sensor name="${name}_depth" type="depth"> -->
-      <sensor name="${name}_depth" type="rgbd_camera">
-        <camera name="${name}">
+        <update_rate>15.0</update_rate>
+        <topic>${name}_depth</topic>
+        <gz_frame_id>${name}_depth</gz_frame_id>
+        <camera name="${name}_depth">
           <camera_info_topic>${name}_depth/camera_info</camera_info_topic>
             <horizontal_fov>1.57</horizontal_fov>
             <image>
-              <width>${depth_width}</width>
-              <height>${depth_height}</height>
+              <width>640</width>
+              <height>480</height>
+              <format>B8G8R8</format>
             </image>
           <clip>
@@ -175,9 +134,4 @@
           </noise>
         </camera>
-        <always_on>true</always_on>
-        <update_rate>30</update_rate>
-        <visualize>false</visualize>
-        <topic>${name}_depth_to_color/image_raw</topic>
-        <gz_frame_id>${name}_depth_optical_frame</gz_frame_id>
       </sensor>
     </gazebo>

File: parc_robot_description/urdf/gz_control.xacro (robot description, xacro)
@@ -15,5 +15,5 @@
         <!-- Control gains and limits (optional) -->
         <!-- <max_velocity>3.0</max_velocity>  -->
-        <max_velocity>1.0</max_velocity>
+        <max_velocity>0.5</max_velocity>
         <max_linear_acceleration>1</max_linear_acceleration>
         <min_linear_acceleration>-1</min_linear_acceleration>
@@ -38,5 +38,5 @@
         <joint_name>right_wheel_joint</joint_name>
     </plugin>
-    <!-- Pose publisher publishes the pose on gz topic /parc_robot/pose
+    <!-- Pose publisher publishes the pose on gz topic /sitoe_robot/pose
     Confirm by listing topics with gz topic -l. Bridge topic data with ROS in
     the gz_bridge.yaml file -->

File: parc_robot_description/urdf/imu.xacro (robot description, xacro)
@@ -9,73 +9,73 @@
   <gazebo reference="imu_link">
     <sensor name="imu_sensor" type="imu">
-    <pose>0 0 0 0 0 0</pose>
-    <gravity>true</gravity>
-    <always_on>true</always_on>
-    <update_rate>100</update_rate>
-    <gz_frame_id>imu_link</gz_frame_id>
-    <visualize>true</visualize>
-    <topic>imu</topic>
-    <imu>
-      <angular_velocity>
-        <x>
-          <noise type="gaussian">
-            <mean>0.0</mean>
-            <stddev>2e-4</stddev>
-          </noise>
-        </x>
-        <y>
-          <noise type="gaussian">
-            <mean>0.0</mean>
-            <stddev>2e-4</stddev>
-          </noise>
-        </y>
-        <z>
-          <noise type="gaussian">
-            <mean>0.0</mean>
-            <stddev>2e-4</stddev>
-          </noise>
-        </z>
-      </angular_velocity>
-      <linear_acceleration>
-        <x>
-          <noise type="gaussian">
-            <mean>0.0</mean>
-            <stddev>1.7e-2</stddev>
-          </noise>
-        </x>
-        <y>
-          <noise type="gaussian">
-            <mean>0.0</mean>
-            <stddev>1.7e-2</stddev>
-          </noise>
-        </y>
-        <z>
-          <noise type="gaussian">
-            <mean>0.0</mean>
-            <stddev>1.7e-2</stddev>
-          </noise>
-        </z>
-      </linear_acceleration>
-      <orientation>
-        <x>
-          <noise type="gaussian">
-            <mean>0.0</mean>
-            <stddev>2e-3</stddev>
-           </noise>
-        </x>
-        <y>
-          <noise type="gaussian">
-            <mean>0.0</mean>
-            <stddev>2e-3</stddev>
-          </noise>
-        </y>
-        <z>
-          <noise type="gaussian">
-            <mean>0.0</mean>
-            <stddev>2e-3</stddev>
-          </noise>
-        </z>
-      </orientation>
-    </imu>
+      <pose>0 0 0 0 0 0</pose>
+      <gravity>true</gravity>
+      <always_on>true</always_on>
+      <update_rate>100</update_rate>
+      <gz_frame_id>imu_link</gz_frame_id>
+      <visualize>true</visualize>
+      <topic>imu</topic>
+      <imu>
+        <angular_velocity>
+          <x>
+            <noise type="gaussian">
+              <mean>0.0</mean>
+              <stddev>2e-4</stddev>
+            </noise>
+          </x>
+          <y>
+            <noise type="gaussian">
+              <mean>0.0</mean>
+              <stddev>2e-4</stddev>
+            </noise>
+          </y>
+          <z>
+            <noise type="gaussian">
+              <mean>0.0</mean>
+              <stddev>2e-4</stddev>
+            </noise>
+          </z>
+        </angular_velocity>
+        <linear_acceleration>
+          <x>
+            <noise type="gaussian">
+              <mean>0.0</mean>
+              <stddev>1.7e-2</stddev>
+            </noise>
+          </x>
+          <y>
+            <noise type="gaussian">
+              <mean>0.0</mean>
+              <stddev>1.7e-2</stddev>
+            </noise>
+          </y>
+          <z>
+            <noise type="gaussian">
+              <mean>0.0</mean>
+              <stddev>1.7e-2</stddev>
+            </noise>
+          </z>
+        </linear_acceleration>
+        <orientation>
+          <x>
+            <noise type="gaussian">
+              <mean>0.0</mean>
+              <stddev>2e-3</stddev>
+             </noise>
+          </x>
+          <y>
+            <noise type="gaussian">
+              <mean>0.0</mean>
+              <stddev>2e-3</stddev>
+            </noise>
+          </y>
+          <z>
+            <noise type="gaussian">
+              <mean>0.0</mean>
+              <stddev>2e-3</stddev>
+            </noise>
+          </z>
+        </orientation>
+      </imu>
     </sensor>
   </gazebo>

File: parc_robot_description/urdf/ros2_control.xacro (robot description, xacro)
@@ -1,3 +1,30 @@
 <?xml version="1.0" ?>
 <robot xmlns:xacro="http://www.ros.org/wiki/xacro">
+<ros2_control name="GazeboSimSystem" type="system">
+    <hardware>
+      <plugin>gz_ros2_control/GazeboSimSystem</plugin>
+    </hardware>
+    <joint name='left_wheel_joint'>
+      <command_interface name='velocity'>
+        <param name='min'>-1</param>
+        <param name='max'>1</param>
+      </command_interface>
+      <state_interface name='velocity'/>
+      <state_interface name='position'/>
+    </joint>
+    <joint name='right_wheel_joint'>
+      <command_interface name='velocity'>
+        <param name='min'>-1</param>
+        <param name='max'>1</param>
+      </command_interface>
+      <state_interface name='velocity'/>
+      <state_interface name='position'/>
+    </joint>
+  </ros2_control>
+  <gazebo>
+    <plugin filename="libgz_ros2_control-system.so" name="gz_ros2_control::GazeboSimROS2ControlPlugin">
+       <parameters>$(find parc_robot_bringup)/config/controllers.yaml</parameters>
+       <parameters>$(find parc_robot_bringup)/config/gazebo_ros2_ctl_use_sim.yaml</parameters>
+    </plugin>
+  </gazebo>
 </robot>

File: parc_robot_description/urdf/rplidar_c1.xacro (robot description, xacro)
@@ -31,5 +31,4 @@
       <topic>scan</topic>
       <gz_frame_id>lidar_link</gz_frame_id>
-      <!-- <lidar> -->
       <ray>
         <scan>
@@ -51,5 +50,4 @@
         </noise>
       </ray>
-      <!-- </lidar> -->
     </sensor>
   </gazebo>
