Commit message: Update robot xacro files

File: parc_robot_description/urdf/sitoe_core.xacro (robot description, xacro)
@@ -22,141 +22,8 @@
       <origin rpy="${pi/2} 0 0" xyz="0.0 0.0 0.0"/>
       <geometry>
-        <mesh filename="package://parc_robot_description/meshes/mainbody.dae"/>
-      </geometry>
-    </visual>
-    <visual>
-      <origin rpy="${pi/2} 0 0" xyz="0.0 0.0 0.0"/>
-      <geometry>
-        <mesh filename="package://parc_robot_description/meshes/mainbody001.dae"/>
-      </geometry>
-    </visual>
-    <visual>
-      <origin rpy="${pi/2} 0 0" xyz="0.0 0.0 0.0"/>
-      <geometry>
-        <mesh filename="package://parc_robot_description/meshes/camerasupport.dae"/>
-      </geometry>
-    </visual>
-    <visual>
-      <origin rpy="${pi/2} 0 0" xyz="0.0 0.0 0.0"/>
-      <geometry>
-        <mesh filename="package://parc_robot_description/meshes/camsupport_2.dae"/>
-      </geometry>
-    </visual>
-    <visual>
-      <origin rpy="${pi/2} 0 0" xyz="0.0 0.0 0.0"/>
-      <geometry>
-        <mesh filename="package://parc_robot_description/meshes/emergencybutton.dae"/>
-      </geometry>
-    </visual>
-    <visual>
-      <origin rpy="${pi/2} 0 0" xyz="0.0 0.0 0.0"/>
-      <geometry>
-        <mesh filename="package://parc_robot_description/meshes/trappe.dae"/>
-      </geometry>
-    </visual>
-    <visual>
-      <origin rpy="${pi/2} 0 0" xyz="0.0 0.0 0.0"/>
-      <geometry>
-        <mesh filename="package://parc_robot_description/meshes/hingea.dae"/>
-      </geometry>
-    </visual>
-    <visual>
-      <origin rpy="${pi/2} 0 0" xyz="0.0 0.0 0.0"/>
-      <geometry>
-        <mesh filename="package://parc_robot_description/meshes/hingeb.dae"/>
-      </geometry>
-    </visual>
-    <visual>
-      <origin rpy="${pi/2} 0 0" xyz="0.0 0.0 0.0"/>
-      <geometry>
-        <mesh filename="package://parc_robot_description/meshes/cameracase.dae"/>
-      </geometry>
-    </visual>
-    <visual>
-      <origin rpy="${pi/2} 0 0" xyz="0.0 0.0 0.0"/>
-      <geometry>
-        <mesh filename="package://parc_robot_description/meshes/arducamcover.dae"/>
-      </geometry>
-    </visual>
-    <visual>
-      <origin rpy="${pi/2} 0 0" xyz="0.0 0.0 0.0"/>
-      <geometry>
-        <mesh filename="package://parc_robot_description/meshes/arducamsupport_r.dae"/>
-      </geometry>
-    </visual>
-    <visual>
-      <origin rpy="${pi/2} 0 0" xyz="0.0 0.0 0.0"/>
-      <geometry>
-        <mesh filename="package://parc_robot_description/meshes/arducamsupport_l.dae"/>
-      </geometry>
-    </visual>
-    <visual>
-      <origin rpy="${pi/2} 0 0" xyz="0.0 0.0 0.0"/>
-      <geometry>
-        <mesh filename="package://parc_robot_description/meshes/arducamsupport_lcover.dae"/>
-      </geometry>
-    </visual>
-    <visual>
-      <origin rpy="${pi/2} 0 0" xyz="0.0 0.0 0.0"/>
-      <geometry>
-        <mesh filename="package://parc_robot_description/meshes/arducamsupport_rcover.dae"/>
-      </geometry>
-    </visual>
-    <visual>
-      <origin rpy="${pi/2} 0 0" xyz="0.0 0.0 0.0"/>
-      <geometry>
-        <mesh filename="package://parc_robot_description/meshes/basecovertop.dae"/>
-      </geometry>
-    </visual>
-    <visual>
-      <origin rpy="${pi/2} 0 0" xyz="0.0 0.0 0.0"/>
-      <geometry>
-        <mesh filename="package://parc_robot_description/meshes/backlid.dae"/>
-      </geometry>
-    </visual>
-    <visual>
-      <origin rpy="${pi/2} 0 0" xyz="0.0 0.0 0.0"/>
-      <geometry>
-        <mesh filename="package://parc_robot_description/meshes/backlid001.dae"/>
-      </geometry>
-    </visual>
-    <visual>
-      <origin rpy="${pi/2} 0 0" xyz="0.0 0.0 0.0"/>
-      <geometry>
-        <mesh filename="package://parc_robot_description/meshes/base.dae"/>
-      </geometry>
-    </visual>
-    <visual>
-      <origin rpy="${pi/2} 0 0" xyz="0.0 0.0 0.0"/>
-      <geometry>
-        <mesh filename="package://parc_robot_description/meshes/base001.dae"/>
-      </geometry>
-    </visual>
-    <visual>
-      <origin rpy="${pi/2} 0 0" xyz="0.0 0.0 0.0"/>
-      <geometry>
-        <mesh filename="package://parc_robot_description/meshes/formedhexscrew_am_b18_2_3_2mformedhexscrewm12x1_75x5030wn.dae"/>
-      </geometry>
-    </visual>
-    <visual>
-      <origin rpy="${pi/2} 0 0" xyz="0.0 0.0 0.0"/>
-      <geometry>
-        <mesh filename="package://parc_robot_description/meshes/hexnutjam_am_b18_2_4_5mhexjamnutm12x1_75dn.dae"/>
-      </geometry>
-    </visual>
-    <visual>
-      <origin rpy="${pi/2} 0 0" xyz="0.0 0.0 0.0"/>
-      <geometry>
-        <mesh filename="package://parc_robot_description/meshes/hexnutjam_am_b18_2_4_5mhexjamnutm14x2dn.dae"/>
-      </geometry>
-    </visual>
-    <visual>
-      <origin rpy="${pi/2} 0 0" xyz="0.0 0.0 0.0"/>
-      <geometry>
-        <mesh filename="package://parc_robot_description/meshes/formedhexscrew_am_b18_2_3_2mformedhexscrewm14x2_0x1616wn.dae"/>
+        <mesh filename="package://parc_robot_description/meshes/sitoe_chassis.dae"/>
       </geometry>
     </visual>
     <collision>
-      <!--col__base_link__col_robot_chassis__BoundBox/col_robot_chassis__BoundBox.-->
       <origin rpy="${pi/2} 0 0" xyz="0.0 0.0454341 0.67537"/>
       <geometry>
@@ -165,35 +32,27 @@
     </collision>
     <xacro:box_inertia mass="15.0" length="${base_length}" width="${base_width}" height="${base_height}">
-      <origin xyz="0.105 0 0.0175" rpy="0 0 0"/>
+      <origin rpy="${pi/2} 0 0" xyz="0.0 0 0.67537"/>
     </xacro:box_inertia>
   </link>
+  <!-- Robot chassis bumper -->
+  <gazebo reference="base_link">
+    <sensor name="base_collision_sensor" type="contact">
+      <contact>
+        <collision>base_footprint_fixed_joint_lump__base_link_collision</collision>
+        <topic>base_collisions</topic>
+      </contact>
+      <always_on>true</always_on>
+      <update_rate>5</update_rate>
+    </sensor>
+  </gazebo>
   <!-- Right wheel -->
   <link name="right_wheel_link">
     <visual>
-      <origin rpy="0 -${pi/2} 0" xyz="0.069 0.01075 0.0267"/>
+      <origin rpy="0 -${pi/2} 0" xyz="0.0956 -0.0435 0.1965"/> <!-- up, forward, sideways-->
       <geometry>
-        <mesh filename="package://parc_robot_description/meshes/botwheel_housing1.dae"/>
-      </geometry>
-    </visual>
-    <visual>
-      <origin rpy="0 -${pi/2} 0" xyz="0.069 0.01075 0.0267"/>
-      <geometry>
-        <mesh filename="package://parc_robot_description/meshes/botwheel_centerpin.dae"/>
-      </geometry>
-    </visual>
-    <visual>
-      <origin rpy="0 -${pi/2} 0" xyz="0.069 0.01075 0.0267"/>
-      <geometry>
-        <mesh filename="package://parc_robot_description/meshes/botwheel_housing2.dae"/>
-      </geometry>
-    </visual>
-    <visual>
-      <origin rpy="0 -${pi/2} 0" xyz="0.069 0.01075 0.0267"/>
-      <geometry>
-        <mesh filename="package://parc_robot_description/meshes/botwheel_tyre.dae"/>
+        <mesh filename="package://parc_robot_description/meshes/right_wheel.dae"/>
       </geometry>
     </visual>
     <collision>
-      <!--col__right_wheel_link__col_right_wheel__BoundCylinder/col_right_wheel__BoundCylinder.-->
       <origin rpy="0 0 0" xyz="0.0 0.0 0.0"/>
       <geometry>
@@ -202,11 +61,23 @@
     </collision>
     <xacro:cylinder_inertia mass="${wheel_mass}" length="${wheel_height}" radius="${wheel_radius}">
-      <origin xyz="0.0 0.0 0.0" rpy="0 0 0"/>
+      <origin rpy="0 0 0" xyz="0.0 0.0 0.0"/>
     </xacro:cylinder_inertia>
   </link>
+  <!-- Right wheel bumper -->
+  <gazebo reference="right_wheel_link">
+    <sensor name="right_wheel_collision_sensor" type="contact">
+      <contact>
+        <collision>right_wheel_link_collision</collision>
+        <topic>right_wheel_collisions</topic>
+      </contact>
+      <always_on>true</always_on>
+      <update_rate>5</update_rate>
+    </sensor>
+  </gazebo>
   <joint name="right_wheel_joint" type="continuous">
     <parent link="base_link"/>
     <child link="right_wheel_link"/>
-    <origin rpy="0 ${pi/2} 0" xyz="-0.19649 -0.095 0.0476"/>
+    <!-- <origin rpy="0 ${pi/2} 0" xyz="-0.19649 -0.095 0.0476"/> -->
+    <origin rpy="0 ${pi/2} 0" xyz="-0.19649 -0.0945 0.0476"/>
     <axis xyz="0 0 1"/>
   </joint>
@@ -214,29 +85,10 @@
   <link name="left_wheel_link">
     <visual>
-      <origin rpy="0 -${pi/2} 0" xyz="0.069 0.01075 0.0267"/>
+      <origin rpy="0 ${pi/2} 0" xyz="-0.0935 -0.044 0.1965"/>
       <geometry>
-        <mesh filename="package://parc_robot_description/meshes/botwheel_housing001.dae"/>
-      </geometry>
-    </visual>
-    <visual>
-      <origin rpy="0 -${pi/2} 0" xyz="0.069 0.01075 0.0267"/>
-      <geometry>
-        <mesh filename="package://parc_robot_description/meshes/botwheel_centerpin001.dae"/>
-      </geometry>
-    </visual>
-    <visual>
-      <origin rpy="0 -${pi/2} 0" xyz="0.069 0.01075 0.0267"/>
-      <geometry>
-        <mesh filename="package://parc_robot_description/meshes/botwheel_housing002.dae"/>
-      </geometry>
-    </visual>
-    <visual>
-      <origin rpy="0 -${pi/2} 0" xyz="0.069 0.01075 0.0267"/>
-      <geometry>
-        <mesh filename="package://parc_robot_description/meshes/botwheel_tyre001.dae"/>
+        <mesh filename="package://parc_robot_description/meshes/left_wheel.dae"/>
       </geometry>
     </visual>
     <collision>
-      <!--col__left_wheel_link__col_left_wheel__BoundCylinder/col_left_wheel__BoundCylinder.-->
       <origin rpy="0 0 0" xyz="0.0 0.0 0.0"/>
       <geometry>
@@ -245,7 +97,18 @@
     </collision>
     <xacro:cylinder_inertia mass="${wheel_mass}" length="${wheel_height}" radius="${wheel_radius}">
-      <origin xyz="0.0 0.0 0.0" rpy="0 0 0"/>
+      <origin rpy="0 0 0" xyz="0.0 0.0 0.0"/>
     </xacro:cylinder_inertia>
   </link>
+  <!-- Left wheel bumper -->
+  <gazebo reference="left_wheel_link">
+    <sensor name="left_wheel_collision_sensor" type="contact">
+      <contact>
+        <collision>left_wheel_link_collision</collision>
+        <topic>left_wheel_collisions</topic>
+      </contact>
+      <always_on>true</always_on>
+      <update_rate>5</update_rate>
+    </sensor>
+  </gazebo>
   <joint name="left_wheel_joint" type="continuous">
     <parent link="base_link"/>
@@ -269,5 +132,5 @@
     </collision>
     <xacro:sphere_inertia mass="0.45" radius="${caster_wheel_radius}">
-      <origin xyz="0.0 0.0 0.0" rpy="0 0 0"/>
+      <origin rpy="0 0 0" xyz="0.0 0.0 0.0"/>
     </xacro:sphere_inertia>
   </link>
@@ -277,4 +140,24 @@
     <origin rpy="0 0 -${pi/2}" xyz="0.0 0.133 0.0"/>
   </joint>
-  <!-- Add friction for gazebo -->
+  <!-- Friction -->
+  <gazebo reference="base_link">
+    <mu1>0.2</mu1>
+    <mu2>0.2</mu2>
+  </gazebo>
+  <gazebo reference="right_wheel_link">
+    <mu1>0.9</mu1>
+    <mu2>0.7</mu2>
+    <kp>10000000.0</kp>
+    <kd>0.0</kd>
+    <kd>1.0</kd>
+    <minDepth>0.001</minDepth>
+  </gazebo>
+  <gazebo reference="left_wheel_link">
+    <mu1>0.9</mu1>
+    <mu2>0.7</mu2>
+    <kp>10000000.0</kp>
+    <kd>0.0</kd>
+    <kd>1.0</kd>
+    <minDepth>0.001</minDepth>
+  </gazebo>
 </robot>

Commit message: Update xacro and config files

File: parc_robot_description/urdf/d435.xacro (robot description, xacro)
@@ -1,5 +1,5 @@
 <?xml version="1.0" ?>
 <robot xmlns:xacro="http://www.ros.org/wiki/xacro">
-  <xacro:macro name="d435" params="name *origin *mesh">
+  <xacro:macro name="d435" params="name parent *origin *mesh">
   <!-- D435 camera sensor offsets -->
   <xacro:property name="d435_cam_depth_to_infra1_offset" value="0.0"/>
@@ -17,5 +17,5 @@
     <!-- D435 camera joint -->
     <joint name="${name}_joint" type="fixed">
-      <parent link="base_link"/>
+      <parent link="${parent}"/>
       <child link="${name}_link"/>
       <xacro:if value="${name=='top_camera'}">

File: parc_robot_description/urdf/depth_cameras.xacro (robot description, xacro)
@@ -3,10 +3,10 @@
   <xacro:include filename="d435.xacro"/>
   <!-- Top D435 camera -->
-  <xacro:d435 name="top_camera">
+  <xacro:d435 name="top_camera" parent="top_chassis_link">
     <origin rpy="${pi/2} 0 ${pi/2}" xyz="0.0525 0.0 -0.9745"/>
     <mesh filename="package://parc_robot_description/meshes/realsense_d435_top.dae"/>
   </xacro:d435>
   <!-- Bottom D435 camera -->
-  <xacro:d435 name="bottom_camera">
+  <xacro:d435 name="bottom_camera" parent="base_link">
     <origin rpy="${pi/6} 0 ${pi/2}" xyz="0.433 0.0 -0.34"/>
     <mesh filename="package://parc_robot_description/meshes/realsense_d435_bottom.dae"/>

File: parc_robot_description/urdf/rplidar_c1.xacro (robot description, xacro)
@@ -25,7 +25,7 @@
   <gazebo reference="lidar_link">
     <sensor name="rplidar_c1" type="gpu_lidar">
-      <pose>0 0 0 0 0 0</pose>
+      <pose>0 0 0.01 0 -${pi/72} 0</pose>
       <always_on>true</always_on>
-      <visualize>false</visualize>
+      <visualize>true</visualize>
       <update_rate>10</update_rate>
       <topic>scan</topic>

File: parc_robot_description/urdf/sitoe_core.xacro (robot description, xacro)
@@ -2,8 +2,11 @@
 <robot name="sitoe" xmlns:xacro="http://www.ros.org/wiki/xacro">
   <xacro:include filename="inertial_macros.xacro"/>
-  <!-- Robot's base properties -->
-  <xacro:property name="base_length" value="0.4437"/>
-  <xacro:property name="base_width" value="1.2714"/>
-  <xacro:property name="base_height" value="0.4858"/>
+  <!-- Robot's chassis properties -->
+  <xacro:property name="top_chassis_length" value="0.4437"/>
+  <xacro:property name="top_chassis_width" value="1.248"/>
+  <xacro:property name="top_chassis_height" value="0.4858"/>
+  <xacro:property name="bottom_chassis_length" value="0.4437"/>
+  <xacro:property name="bottom_chassis_width" value="0.03785"/>
+  <xacro:property name="bottom_chassis_height" value="0.3737"/>
   <!-- Robot's wheel properties -->
   <xacro:property name="wheel_radius" value="0.086"/>
@@ -11,4 +14,5 @@
   <xacro:property name="wheel_mass" value="2.2"/>
   <xacro:property name="caster_wheel_radius" value="0.0508"/>
+  <!-- Base footprint -->
   <link name="base_footprint"/>
   <joint name="base_joint" type="fixed">
@@ -17,20 +21,20 @@
     <origin rpy="0 0 ${pi/2}" xyz="0.0 0.0 0.0381"/>
   </joint>
-  <!-- Robot chassis -->
+  <!-- Base link/bottom chassis -->
   <link name="base_link">
     <visual>
       <origin rpy="${pi/2} 0 0" xyz="0.0 0.0 0.0"/>
       <geometry>
-        <mesh filename="package://parc_robot_description/meshes/sitoe_chassis.dae"/>
-      </geometry>
-    </visual>
-    <collision>
-      <origin rpy="${pi/2} 0 0" xyz="0.0 0.0454341 0.67537"/>
-      <geometry>
-        <box size="${base_length} ${base_width} ${base_height}"/>
-      </geometry>
-    </collision>
-    <xacro:box_inertia mass="15.0" length="${base_length}" width="${base_width}" height="${base_height}">
-      <origin rpy="${pi/2} 0 0" xyz="0.0 0 0.67537"/>
+        <mesh filename="package://parc_robot_description/meshes/sitoe_chassis_bottom.dae"/>
+      </geometry>
+    </visual>
+    <collision>
+      <origin rpy="${pi/2} 0 0" xyz="0.0 0.0 0.0535"/>
+      <geometry>
+        <box size="${bottom_chassis_length} ${bottom_chassis_width} ${bottom_chassis_height}"/>
+      </geometry>
+    </collision>
+    <xacro:box_inertia mass="7.50" length="${bottom_chassis_length}" width="${bottom_chassis_width}" height="${bottom_chassis_height}">
+      <origin rpy="${pi/2} 0 0" xyz="0.0 0.0 0.0535"/>
     </xacro:box_inertia>
   </link>
@@ -46,8 +50,43 @@
     </sensor>
   </gazebo>
+  <!-- Top chassis -->
+  <link name="top_chassis_link">
+    <visual>
+      <origin rpy="${pi/2} 0 0" xyz="0.0 0.0 0.0"/>
+      <geometry>
+        <mesh filename="package://parc_robot_description/meshes/sitoe_chassis_top.dae"/>
+      </geometry>
+    </visual>
+    <collision>
+      <origin rpy="${pi/2} 0 0" xyz="0.0 0.0454341 0.68679"/>
+      <geometry>
+        <box size="${top_chassis_length} ${top_chassis_width} ${top_chassis_height}"/>
+      </geometry>
+    </collision>
+    <xacro:box_inertia mass="7.50" length="${top_chassis_length}" width="${top_chassis_width}" height="${top_chassis_height}">
+      <origin rpy="${pi/2} 0 0" xyz="0.0 0.0454341 0.68679"/>
+    </xacro:box_inertia>
+  </link>
+  <!-- Top chassis bumper -->
+  <gazebo reference="top_chassis_link">
+    <sensor name="top_chassis_collision_sensor" type="contact">
+      <contact>
+        <collision>base_footprint_fixed_joint_lump__top_chassis_link_collision_2</collision>
+        <topic>top_chassis_collisions</topic>
+      </contact>
+      <always_on>true</always_on>
+      <update_rate>5</update_rate>
+    </sensor>
+  </gazebo>
+  <joint name="chassis_joint" type="fixed">
+    <parent link="base_link"/>
+    <child link="top_chassis_link"/>
+    <origin rpy="0 0 0" xyz="0.0 0.0 0.0"/>
+  </joint>
   <!-- Right wheel -->
   <link name="right_wheel_link">
     <visual>
-      <origin rpy="0 -${pi/2} 0" xyz="0.0956 -0.0435 0.1965"/> <!-- up, forward, sideways-->
+      <origin rpy="0 -${pi/2} 0" xyz="0.0956 -0.0435 0.19096"/> <!-- up, forward, sideways-->
+      <!-- <origin rpy="0 -${pi/2} 0" xyz="0.0956 -0.0435 0.1965"/> -->
       <geometry>
         <mesh filename="package://parc_robot_description/meshes/right_wheel.dae"/>
@@ -55,5 +94,5 @@
     </visual>
     <collision>
-      <origin rpy="0 0 0" xyz="0.0 0.0 0.0"/>
+      <origin rpy="0 0 0" xyz="0.0 0.0 -0.006"/>
       <geometry>
         <cylinder length="${wheel_height}" radius="${wheel_radius}"/>
@@ -61,5 +100,5 @@
     </collision>
     <xacro:cylinder_inertia mass="${wheel_mass}" length="${wheel_height}" radius="${wheel_radius}">
-      <origin rpy="0 0 0" xyz="0.0 0.0 0.0"/>
+      <origin rpy="0 0 0" xyz="0.0 0.0 -0.006"/>
     </xacro:cylinder_inertia>
   </link>
@@ -78,6 +117,6 @@
     <parent link="base_link"/>
     <child link="right_wheel_link"/>
-    <!-- <origin rpy="0 ${pi/2} 0" xyz="-0.19649 -0.095 0.0476"/> -->
-    <origin rpy="0 ${pi/2} 0" xyz="-0.19649 -0.0945 0.0476"/>
+    <origin rpy="0 ${pi/2} 0" xyz="-0.19649 -0.095 0.0476"/>
+    <!-- <origin rpy="0 ${pi/2} 0" xyz="-0.19649 -0.0945 0.0476"/> -->
     <axis xyz="0 0 1"/>
   </joint>
@@ -85,5 +124,5 @@
   <link name="left_wheel_link">
     <visual>
-      <origin rpy="0 ${pi/2} 0" xyz="-0.0935 -0.044 0.1965"/>
+      <origin rpy="0 ${pi/2} 0" xyz="-0.0956 -0.0435 0.19096"/> <!-- up, forward, sideways-->
       <geometry>
         <mesh filename="package://parc_robot_description/meshes/left_wheel.dae"/>
@@ -91,5 +130,5 @@
     </visual>
     <collision>
-      <origin rpy="0 0 0" xyz="0.0 0.0 0.0"/>
+      <origin rpy="0 0 0" xyz="0.0 0.0 -0.006"/>
       <geometry>
         <cylinder length="${wheel_height}" radius="${wheel_radius}"/>
@@ -97,5 +136,5 @@
     </collision>
     <xacro:cylinder_inertia mass="${wheel_mass}" length="${wheel_height}" radius="${wheel_radius}">
-      <origin rpy="0 0 0" xyz="0.0 0.0 0.0"/>
+      <origin rpy="0 0 0" xyz="0.0 0.0 -0.006"/>
     </xacro:cylinder_inertia>
   </link>
@@ -141,5 +180,5 @@
   </joint>
   <!-- Friction -->
-  <gazebo reference="base_link">
+  <gazebo reference="caster_wheel_link">
     <mu1>0.2</mu1>
     <mu2>0.2</mu2>

File: parc_robot_description/urdf/sitoe_robot.urdf (robot description, URDF)
Before this commit: robot sitoe_robot, 23 links, 22 joints
Links:
- added link bottom_camera_depth
- added link top_camera_depth
- added link top_chassis_link, mass 7.5; collision box size=0.4437 1.248 0.4858; visual mesh filename=package://parc_robot_description/meshes/sitoe_chassis_top.d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
- link base_link: mass 15.0 -> 7.5; geometry collision box size=0.4437 0.03785 0.3737; visual mesh filename=package://parc_robot_description/meshes/sitoe_chassis_botto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
Joints:
- added joint bottom_camera_depth_optical_joint: type fixed, parent bottom_camera_depth, child bottom_camera_depth_optical_frame, origin xyz=0.0 0.0 0.0 rpy=-1.5707963267948966 0 -1.5707963267948966
- added joint chassis_joint: type fixed, parent base_link, child top_chassis_link, origin xyz=0.0 0.0 0.0 rpy=0 0 0
- added joint top_camera_depth_optical_joint: type fixed, parent top_camera_depth, child top_camera_depth_optical_frame, origin xyz=0.0 0.0 0.0 rpy=-1.5707963267948966 0 -1.5707963267948966
- joint bottom_camera_depth_joint: child bottom_camera_depth_optical_frame -> bottom_camera_depth; origin xyz=0.0 0.0 0.0 rpy=-1.5707963267948966 0 -1.5707963267948966 -> xyz=0 0 0 rpy=0 0 0
- joint bottom_camera_infra1_optical_joint: origin xyz=0 0 0 rpy=-1.5707963267948966 0 -1.5707963267948966 -> xyz=0.0 0.0 0.0 rpy=-1.5707963267948966 0 -1.5707963267948966
- joint bottom_camera_infra2_optical_joint: origin xyz=0 0 0 rpy=-1.5707963267948966 0 -1.5707963267948966 -> xyz=0.0 0.0 0.0 rpy=-1.5707963267948966 0 -1.5707963267948966
- joint top_camera_depth_joint: child top_camera_depth_optical_frame -> top_camera_depth; origin xyz=0.0 0.0 0.0 rpy=-1.5707963267948966 0 -1.5707963267948966 -> xyz=0 0 0 rpy=0 0 0
- joint top_camera_infra1_optical_joint: origin xyz=0 0 0 rpy=-1.5707963267948966 0 -1.5707963267948966 -> xyz=0.0 0.0 0.0 rpy=-1.5707963267948966 0 -1.5707963267948966
- joint top_camera_infra2_optical_joint: origin xyz=0 0 0 rpy=-1.5707963267948966 0 -1.5707963267948966 -> xyz=0.0 0.0 0.0 rpy=-1.5707963267948966 0 -1.5707963267948966
- joint top_camera_joint: parent base_link -> top_chassis_link
